Commit message: joystick control launch file

File: description/properties.xacro (robot description, xacro)
@@ -14,3 +14,17 @@
         <color rgba= "0 0 0 1"/>
     </material>
+    <gazebo reference="chassis">
+        <material>Gazebo/White</material>
+    </gazebo>
+    <gazebo reference="left_wheel">
+        <material>Gazebo/Blue</material>
+    </gazebo>
+    <gazebo reference="right_wheel">
+        <material>Gazebo/Blue</material>
+    </gazebo>
+    <gazebo reference="caster_wheel">
+        <material>Gazebo/Black</material>
+        <mu1 value = "0.001" />
+        <mu2 value = "0.001" />
+    </gazebo>
 </robot>

File: description/robot.urdf.xacro (robot description, xacro)
@@ -3,3 +3,4 @@
     <xacro:include filename="properties.xacro"/>
     <xacro:include filename="robot_core.xacro"/>
+    <xacro:include filename="gazebo_control.xacro"/>
 </robot>

Commit message: Lidar

File: description/properties.xacro (robot description, xacro)
@@ -4,4 +4,7 @@
     <material name="white">
         <color rgba= "1 1 1 1"/>
+    </material>
+    <material name="red">
+        <color rgba= "1 0 0 1"/>
     </material>
     <material name="orange">

File: description/robot.urdf.xacro (robot description, xacro)
@@ -4,3 +4,4 @@
     <xacro:include filename="robot_core.xacro"/>
     <xacro:include filename="gazebo_control.xacro"/>
+    <xacro:include filename="lidar.xacro"/>
 </robot>

Commit message: IMU+twist_mux

File: description/properties.xacro (robot description, xacro)
@@ -4,7 +4,4 @@
     <material name="white">
         <color rgba= "1 1 1 1"/>
-    </material>
-    <material name="red">
-        <color rgba= "1 0 0 1"/>
     </material>
     <material name="orange">

File: description/robot.urdf.xacro (robot description, xacro)
@@ -5,3 +5,4 @@
     <xacro:include filename="gazebo_control.xacro"/>
     <xacro:include filename="lidar.xacro"/>
+    <xacro:include filename="imu.xacro"/>
 </robot>

File: description/robot_core.xacro (robot description, xacro)
@@ -46,8 +46,8 @@
         </visual>
         <collision>
-            <geometry>
-                <cylinder radius="0.05" length="0.04"/>
-            </geometry>
-        </collision>
+	          <geometry>
+	              <sphere radius="0.05"/>
+	          </geometry>
+	    </collision>
         <xacro:inertial_cylinder mass="0.1" length="0.04" radius="0.05">
             <origin xyz="0 0 0" rpy="0 0 0"/>
@@ -71,5 +71,5 @@
         <collision>
             <geometry>
-                <cylinder radius="0.05" length="0.04"/>
+                <sphere radius="0.05" />
             </geometry>
         </collision>
