Commit message: implementacion TTC, cambios en control que no funcionan bien

File: description/imu.xacro (robot description, xacro)
@@ -3,28 +3,28 @@
     <!-- Define the IMU link -->
     <link name="imu_link">
-    <visual>
-        <geometry>
-        <box size="0.05 0.05 0.05"/>
-        </geometry>
-        <material name="blue">
-        <color rgba="0 0 1 1"/>
-        </material>
-    </visual>
-    <collision>
-        <geometry>
-        <box size="0.05 0.05 0.05"/>
-        </geometry>
-    </collision>
-    <inertial>
-        <mass value="0.1"/>
-        <origin xyz="0 0 0" rpy="0 0 0"/>
-        <inertia ixx="0.0001" ixy="0.0" ixz="0.0" iyy="0.0001" iyz="0.0" izz="0.0001"/>
-    </inertial>
+        <visual>
+            <geometry>
+                <box size="0.05 0.05 0.05"/>
+            </geometry>
+            <material name="blue">
+                <color rgba="0 0 1 1"/>
+            </material>
+        </visual>
+        <collision>
+            <geometry>
+                <box size="0.05 0.05 0.05"/>
+            </geometry>
+        </collision>
+        <inertial>
+            <mass value="0.1"/>
+            <origin xyz="0 0 0" rpy="0 0 0"/>
+            <inertia ixx="0.0001" ixy="0.0" ixz="0.0" iyy="0.0001" iyz="0.0" izz="0.0001"/>
+        </inertial>
     </link>
     <!-- Define the IMU joint -->
     <joint name="imu_joint" type="fixed">
-    <parent link="base_link"/>
-    <child link="imu_link"/>
-    <origin xyz="0 0 0.1" rpy="0 0 0"/>
+        <parent link="base_link"/>
+        <child link="imu_link"/>
+        <origin xyz="0 0 0.1" rpy="0 0 0"/>
     </joint>
     <!-- Define the IMU sensor -->
@@ -35,7 +35,7 @@
             <update_rate>100</update_rate>
             <visualize>1</visualize>
-            <topic>__default_topic__</topic>
+            <topic>/imu</topic>  <!-- Updated topic name -->
             <plugin name='imu_plugin' filename='libgazebo_ros_imu_sensor.so'>
-                <topicName>imu</topicName>
+                <topicName>/imu</topicName>  <!-- Updated topic name -->
                 <bodyName>imu_link</bodyName>
                 <updateRateHZ>10.0</updateRateHZ>
