Commit message: class slam toolbox

File: description/robot_core.xacro (robot description, xacro)
@@ -6,4 +6,12 @@
     <link name="base_link">
     </link>
+    <!-- Example link -->
+    <link name="base_footprint">
+    </link>
+    <joint name="base_footprint_joint" type="fixed">
+        <parent link="base_link"/>
+        <child link="base_footprint"/>
+        <origin xyz="0 0 0"/>
+    </joint>
     <joint name="base_link" type="fixed">
         <parent link="base_link"/>
