Commit message: mapeo funcionando virtual

File: description/gazebo_control.xacro (robot description, xacro)
@@ -11,5 +11,5 @@
             <!-- limits -->
             <max_wheel_torque>200</max_wheel_torque>
-            <max_wheel_acceleration>10.0</max_wheel_acceleration>
+            <max_wheel_acceleration>1.0</max_wheel_acceleration>
             <!-- outputs -->
             <odometry_frame>odom</odometry_frame>

File: description/lidar.xacro (robot description, xacro)
@@ -13,5 +13,5 @@
                 <cylinder radius="0.05" length="0.04"/>
             </geometry>
-            <material name="red"/>
+            <material name="blue"/>
         </visual>
         <collision>
@@ -28,5 +28,5 @@
         <sensor name="laser" type="ray">
             <pose>0 0 0 0 0 0</pose>
-            <visualize>false</visualize>
+            <visualize>true</visualize>
             <update_rate>10</update_rate>
             <ray>

File: description/robot_core.xacro (robot description, xacro)
@@ -3,5 +3,5 @@
     <!-- Example link -->
     <xacro:include filename="inertial_macros.xacro"/>
-    <!-- Example link -->
+   <!-- Example link -->
     <link name="base_link">
     </link>
@@ -9,5 +9,5 @@
     <link name="base_footprint">
     </link>
-    <joint name="base_footprint_joint" type="fixed">
+ <joint name="base_footprint_joint" type="fixed">
         <parent link="base_link"/>
         <child link="base_footprint"/>
@@ -34,5 +34,5 @@
             </geometry>
         </collision>
-        <xacro:inertial_box mass="0.5" x="0.3" y="0.3" z="0.15">
+         <xacro:inertial_box mass="0.5" x="0.3" y="0.3" z="0.15">
             <origin xyz="0.15 0 0.075" rpy="0 0 0"/>
         </xacro:inertial_box>
@@ -54,8 +54,8 @@
         </visual>
         <collision>
-	          <geometry>
-	              <sphere radius="0.05"/>
-	          </geometry>
-	    </collision>
+            <geometry>
+                <cylinder radius="0.05" length="0.04"/>
+            </geometry>
+        </collision>
         <xacro:inertial_cylinder mass="0.1" length="0.04" radius="0.05">
             <origin xyz="0 0 0" rpy="0 0 0"/>
@@ -79,5 +79,5 @@
         <collision>
             <geometry>
-                <sphere radius="0.05" />
+                <cylinder radius="0.05" length="0.04"/>
             </geometry>
         </collision>
@@ -109,3 +109,17 @@
         </xacro:inertial_sphere>
     </link>
+    <gazebo reference="chassis">
+        <material>Gazebo/White</material>
+    </gazebo>
+    <gazebo reference="left_wheel">
+        <material>Gazebo/Blue</material>
+    </gazebo>
+    <gazebo reference="right_wheel">
+        <material>Gazebo/Blue</material>
+    </gazebo>
+    <gazebo reference="caster_wheel">
+        <material>Gazebo/Black</material>
+        <mu1 value = "0.001" />
+        <mu2 value = "0.001" />
+    </gazebo>
 </robot>

Commit message: cambios robot ackermann descripcion

File: description/gazebo_control.xacro (robot description, xacro)
@@ -1,21 +1,56 @@
 <?xml version="1.0"?>
-<robot xmlns:xacro="http://www.ros.org/wiki/xacro" >
-    <!-- Example link -->
+<robot xmlns:xacro="http://www.ros.org/wiki/xacro">
     <gazebo>
-        <plugin name="diff_drive" filename="libgazebo_ros_diff_drive.so">
-            <!-- wheels information -->
-            <left_joint>left_wheel_joint</left_joint>
-            <right_joint>right_wheel_joint</right_joint>
-            <wheel_separation>0.35</wheel_separation>
-            <wheel_diameter>0.1</wheel_diameter>
-            <!-- limits -->
-            <max_wheel_torque>200</max_wheel_torque>
-            <max_wheel_acceleration>1.0</max_wheel_acceleration>
-            <!-- outputs -->
-            <odometry_frame>odom</odometry_frame>
-            <robot_base_frame>base_link</robot_base_frame>
+        <!-- Ackermann Drive Plugin Configuration -->
+        <plugin name="gazebo_ros_ackermann_drive" filename="libgazebo_ros_ackermann_drive.so">
+            <!-- ROS Namespace and Remappings -->
+            <ros>
+                <namespace>/</namespace> <!-- Set this to your robot's model name -->
+                <remapping>cmd_vel:=cmd_vel</remapping>
+                <remapping>odom:=odom</remapping>
+            </ros>
+            <!-- Update Rate -->
+            <update_rate>100.0</update_rate>
+            <!-- Wheel Joints -->
+            <front_left_joint>front_left_wheel_joint</front_left_joint>
+            <front_right_joint>front_right_wheel_joint</front_right_joint>
+            <rear_left_joint>rear_left_wheel_joint</rear_left_joint>
+            <rear_right_joint>rear_right_wheel_joint</rear_right_joint>
+            <!-- Steering Joints -->
+            <left_steering_joint>left_steering_joint</left_steering_joint>
+            <right_steering_joint>right_steering_joint</right_steering_joint>
+            <!-- Steering Limits -->
+            <max_steer>0.5</max_steer>
+            <!-- Max Steering Wheel Angle -->
+            <max_steering_angle>7.85</max_steering_angle>
+            <!-- Max Speed -->
+            <max_speed>5.0</max_speed>
+            <!-- PID Tuning -->
+            <left_steering_pid_gain>500 0 50</left_steering_pid_gain>
+            <left_steering_i_range>0 0</left_steering_i_range>
+            <right_steering_pid_gain>500 0 50</right_steering_pid_gain>
+            <right_steering_i_range>0 0</right_steering_i_range>
+            <linear_velocity_pid_gain>300 10 20</linear_velocity_pid_gain>
+            <linear_velocity_i_range>-0.5 0.5</linear_velocity_i_range>
+            <!-- Output -->
             <publish_odom>true</publish_odom>
             <publish_odom_tf>true</publish_odom_tf>
             <publish_wheel_tf>true</publish_wheel_tf>
+            <publish_distance>false</publish_distance>
+            <!-- Frames -->
+            <odometry_frame>odom</odometry_frame>
+            <robot_base_frame>base_link</robot_base_frame>
+        </plugin>
+        <!-- Joint State Publisher Plugin -->
+        <plugin name="joint_state_publisher" filename="libgazebo_ros_joint_state_publisher.so">
+            <robotNamespace>/</robotNamespace> <!-- Set this to your robot's model name -->
+            <publishInterval>0.1</publishInterval>
+            <!-- List all joint names -->
+            <joint_name>front_left_wheel_joint</joint_name>
+            <joint_name>front_right_wheel_joint</joint_name>
+            <joint_name>rear_left_wheel_joint</joint_name>
+            <joint_name>rear_right_wheel_joint</joint_name>
+            <joint_name>left_steering_joint</joint_name>
+            <joint_name>right_steering_joint</joint_name>
         </plugin>
     </gazebo>

File: description/lidar.xacro (robot description, xacro)
@@ -1,24 +1,24 @@
 <?xml version="1.0"?>
 <robot xmlns:xacro="http://www.ros.org/wiki/xacro">
-    <!-- lidar joint -->
+    <!-- Lidar Joint -->
     <joint name="laser_joint" type="fixed">
         <parent link="chassis"/>
         <child link="laser_frame"/>
-        <origin xyz="0.1 0 0.175" rpy="0 0 0"/>
+        <origin xyz="-0.04 0 0.1"/> <!-- 4 cm backward, 13 cm elevation -->
     </joint>
-    <!-- laser_frame -->
+    <!-- Lidar Link -->
     <link name="laser_frame">
         <visual>
             <geometry>
-                <cylinder radius="0.05" length="0.04"/>
+                <cylinder radius="0.05" length="0.025"/> <!-- Example geometry -->
             </geometry>
-            <material name="blue"/>
+            <material name="black"/>
         </visual>
         <collision>
             <geometry>
-                <cylinder radius="0.05" length="0.04"/>
+                <cylinder radius="0.05" length="0.02"/>
             </geometry>
         </collision>
-        <xacro:inertial_cylinder mass="0.1" length="0.04" radius="0.05">
+        <xacro:inertial_cylinder mass="0.1" length="0.02" radius="0.05">
             <origin xyz="0 0 0" rpy="0 0 0"/>
         </xacro:inertial_cylinder>

File: description/robot.urdf.xacro (robot description, xacro)
@@ -5,4 +5,4 @@
     <xacro:include filename="gazebo_control.xacro"/>
     <xacro:include filename="lidar.xacro"/>
-    <xacro:include filename="imu.xacro"/>
+    <!---<xacro:include filename="imu.xacro"/>-->
 </robot>

File: description/robot_core.xacro (robot description, xacro)
@@ -1,125 +1,179 @@
 <?xml version="1.0"?>
 <robot xmlns:xacro="http://www.ros.org/wiki/xacro">
-    <!-- Example link -->
-    <xacro:include filename="inertial_macros.xacro"/>
-   <!-- Example link -->
-    <link name="base_link">
-    </link>
-    <!-- Example link -->
-    <link name="base_footprint">
-    </link>
- <joint name="base_footprint_joint" type="fixed">
-        <parent link="base_link"/>
-        <child link="base_footprint"/>
-        <origin xyz="0 0 0"/>
-    </joint>
-    <joint name="base_link" type="fixed">
-        <parent link="base_link"/>
-        <child link="chassis"/>
-        <origin xyz="-0.1 0 0"/>
-    </joint>
-    <!-- chassis link -->
-    <link name="chassis">
-        <visual>
-            <origin xyz="0.15 0 0.075"/>
-            <geometry>
-                <box size="0.3 0.3 0.15"/>
-            </geometry>
-            <material name="white"/>
-        </visual>
-        <collision>
-            <origin xyz="0.15 0 0.075"/>
-            <geometry>
-                <box size="0.3 0.3 0.15"/>
-            </geometry>
-        </collision>
-         <xacro:inertial_box mass="0.5" x="0.3" y="0.3" z="0.15">
-            <origin xyz="0.15 0 0.075" rpy="0 0 0"/>
-        </xacro:inertial_box>
-    </link>
-    <!-- left wheel joint -->
-    <joint name="left_wheel_joint" type="continuous">
-        <parent link="base_link"/>
-        <child link="left_wheel"/>
-        <origin xyz="0 0.175 0" rpy="-${pi/2} 0 0"/>
-        <axis xyz="0 0 1"/>
-    </joint>
-    <!-- left wheel link -->
-    <link name="left_wheel">
-        <visual>
-            <geometry>
-                <cylinder radius="0.05" length="0.04"/>
-            </geometry>
-            <material name="blue"/>
-        </visual>
-        <collision>
-            <geometry>
-                <cylinder radius="0.05" length="0.04"/>
-            </geometry>
-        </collision>
-        <xacro:inertial_cylinder mass="0.1" length="0.04" radius="0.05">
-            <origin xyz="0 0 0" rpy="0 0 0"/>
-        </xacro:inertial_cylinder>
-    </link>
-    <!-- right wheel joint -->
-    <joint name="right_wheel_joint" type="continuous">
-        <parent link="base_link"/>
-        <child link="right_wheel"/>
-        <origin xyz="0 -0.175 0" rpy="${pi/2} 0 0"/>
-        <axis xyz="0 0 -1"/>
-    </joint>
-    <!-- right wheel link -->
-    <link name="right_wheel">
-        <visual>
-            <geometry>
-                <cylinder radius="0.05" length="0.04"/>
-            </geometry>
-            <material name="blue"/>
-        </visual>
-        <collision>
-            <geometry>
-                <cylinder radius="0.05" length="0.04"/>
-            </geometry>
-        </collision>
-        <xacro:inertial_cylinder mass="0.1" length="0.04" radius="0.05">
-            <origin xyz="0 0 0" rpy="0 0 0"/>
-        </xacro:inertial_cylinder>
-    </link>
-    <!-- caster wheel joint -->
-    <joint name="caster_wheel_joint" type="fixed">
-        <parent link="chassis"/>
-        <child link="caster_wheel"/>
-        <origin xyz="0.24 0 0"/>
-    </joint>
-    <!-- left wheel link -->
-    <link name="caster_wheel">
-        <visual>
-            <geometry>
-                <sphere radius="0.05"/>
-            </geometry>
-            <material name="black"/>
-        </visual>
-        <collision>
-            <geometry>
-                <sphere radius="0.05"/>
-            </geometry>
-        </collision>
-        <xacro:inertial_sphere mass="0.1" radius="0.05">
-            <origin xyz="0 0 0" rpy="0 0 0"/>
-        </xacro:inertial_sphere>
-    </link>
-    <gazebo reference="chassis">
-        <material>Gazebo/White</material>
-    </gazebo>
-    <gazebo reference="left_wheel">
-        <material>Gazebo/Blue</material>
-    </gazebo>
-    <gazebo reference="right_wheel">
-        <material>Gazebo/Blue</material>
-    </gazebo>
-    <gazebo reference="caster_wheel">
-        <material>Gazebo/Black</material>
-        <mu1 value = "0.001" />
-        <mu2 value = "0.001" />
-    </gazebo>
+  <!-- Include Inertial Macros -->
+  <xacro:include filename="inertial_macros.xacro"/>
+  <!-- Base Footprint Joint -->
+  <joint name="base_footprint_joint" type="fixed">
+    <parent link="base_link"/>
+    <child link="base_footprint"/>
+    <origin xyz="0 0 0"/>
+  </joint>
+  <!-- Base Footprint Link -->
+  <link name="base_footprint"/>
+  <!-- Base Link -->
+  <link name="base_link"/>
+  <!-- Base Link to Chassis Joint -->
+  <joint name="base_link_joint" type="fixed">
+    <parent link="base_link"/>
+    <child link="chassis"/>
+    <origin xyz="0 0 0.065"/>
+  </joint>
+  <!-- Chassis Link -->
+  <link name="chassis">
+    <visual>
+      <origin xyz="0 0 0"/>
+      <geometry>
+        <box size="0.24 0.15 0.06"/>
+      </geometry>
+      <material name="white"/>
+    </visual>
+    <collision>
+      <origin xyz="0 0 0"/>
+      <geometry>
+        <box size="0.24 0.15 0.06"/>
+      </geometry>
+    </collision>
+    <xacro:inertial_box mass="3.0" x="0.24" y="0.15" z="0.06">
+      <origin xyz="0 0 0"/>
+    </xacro:inertial_box>
+  </link>
+  <!-- Left Steering Joint -->
+  <joint name="left_steering_joint" type="revolute">
+    <parent link="chassis"/>
+    <child link="left_steering_link"/>
+    <origin xyz="0.12 0.09 -0.0375" rpy="1.5708 0 0"/>
+    <axis xyz="0 1 0"/>
+    <limit lower="-0.5" upper="0.5" effort="1000" velocity="1.0"/>
+  </joint>
+  <!-- Left Steering Link -->
+  <link name="left_steering_link"/>
+  <!-- Front Left Wheel Joint -->
+  <joint name="front_left_wheel_joint" type="continuous">
+    <parent link="left_steering_link"/>
+    <child link="front_left_wheel"/>
+    <origin xyz="0 0 0" rpy="0 0 0"/>
+    <axis xyz="0 0 1"/>
+  </joint>
+  <!-- Front Left Wheel Link -->
+  <link name="front_left_wheel">
+    <visual>
+      <geometry>
+        <cylinder radius="0.0375" length="0.025"/>
+      </geometry>
+      <material name="blue"/>
+    </visual>
+    <collision>
+      <geometry>
+        <cylinder radius="0.0375" length="0.025"/>
+      </geometry>
+    </collision>
+    <xacro:inertial_cylinder mass="0.1" length="0.025" radius="0.0375">
+      <origin xyz="0 0 0"/>
+    </xacro:inertial_cylinder>
+  </link>
+  <!-- Right Steering Joint -->
+  <joint name="right_steering_joint" type="revolute">
+    <parent link="chassis"/>
+    <child link="right_steering_link"/>
+    <origin xyz="0.12 -0.09 -0.0375" rpy="1.5708 0 0"/>
+    <axis xyz="0 1 0"/>
+    <limit lower="-0.5" upper="0.5" effort="1000" velocity="1.0"/>
+  </joint>
+  <!-- Right Steering Link -->
+  <link name="right_steering_link"/>
+  <!-- Front Right Wheel Joint -->
+  <joint name="front_right_wheel_joint" type="continuous">
+    <parent link="right_steering_link"/>
+    <child link="front_right_wheel"/>
+    <origin xyz="0 0 0" rpy="0 0 0"/>
+    <axis xyz="0 0 1"/>
+  </joint>
+  <!-- Front Right Wheel Link -->
+  <link name="front_right_wheel">
+    <visual>
+      <geometry>
+        <cylinder radius="0.0375" length="0.025"/>
+      </geometry>
+      <material name="blue"/>
+    </visual>
+    <collision>
+      <geometry>
+        <cylinder radius="0.0375" length="0.025"/>
+      </geometry>
+    </collision>
+    <xacro:inertial_cylinder mass="0.1" length="0.025" radius="0.0375">
+      <origin xyz="0 0 0"/>
+    </xacro:inertial_cylinder>
+  </link>
+  <!-- Rear Left Wheel Joint -->
+  <joint name="rear_left_wheel_joint" type="continuous">
+    <parent link="chassis"/>
+    <child link="rear_left_wheel"/>
+    <origin xyz="-0.12 0.09 -0.0375" rpy="1.5708 0 0"/>
+    <axis xyz="0 0 1"/>
+  </joint>
+  <!-- Rear Left Wheel Link -->
+  <link name="rear_left_wheel">
+    <visual>
+      <geometry>
+        <cylinder radius="0.0375" length="0.025"/>
+      </geometry>
+      <material name="blue"/>
+    </visual>
+    <collision>
+      <geometry>
+        <cylinder radius="0.0375" length="0.025"/>
+      </geometry>
+    </collision>
+    <xacro:inertial_cylinder mass="0.1" length="0.025" radius="0.0375">
+      <origin xyz="0 0 0"/>
+    </xacro:inertial_cylinder>
+  </link>
+  <!-- Rear Right Wheel Joint -->
+  <joint name="rear_right_wheel_joint" type="continuous">
+    <parent link="chassis"/>
+    <child link="rear_right_wheel"/>
+    <origin xyz="-0.12 -0.09 -0.0375" rpy="1.5708 0 0"/>
+    <axis xyz="0 0 1"/>
+  </joint>
+  <!-- Rear Right Wheel Link -->
+  <link name="rear_right_wheel">
+    <visual>
+      <geometry>
+        <cylinder radius="0.0375" length="0.025"/>
+      </geometry>
+      <material name="blue"/>
+    </visual>
+    <collision>
+      <geometry>
+        <cylinder radius="0.0375" length="0.025"/>
+      </geometry>
+    </collision>
+    <xacro:inertial_cylinder mass="0.1" length="0.025" radius="0.0375">
+      <origin xyz="0 0 0"/>
+    </xacro:inertial_cylinder>
+  </link>
+  <!-- Camera Joint -->
+  <joint name="camera_joint" type="fixed">
+    <parent link="chassis"/>
+    <child link="camera_link"/>
+    <origin xyz="0.10 0 0.04"/>
+  </joint>
+  <!-- Camera Link -->
+  <link name="camera_link">
+    <visual>
+      <geometry>
+        <box size="0.025 0.09 0.02"/>
+      </geometry>
+      <material name="black"/>
+    </visual>
+    <collision>
+      <geometry>
+        <box size="0.025 0.09 0.02"/>
+      </geometry>
+    </collision>
+    <xacro:inertial_box mass="0.05" x="0.025" y="0.09" z="0.02">
+      <origin xyz="0 0 0"/>
+    </xacro:inertial_box>
+  </link>
 </robot>
