Commit message: ros2_control no funcionando

File: description/gazebo_control.xacro (robot description, xacro)
@@ -2,55 +2,36 @@
 <robot xmlns:xacro="http://www.ros.org/wiki/xacro">
     <gazebo>
-        <!-- Ackermann Drive Plugin Configuration -->
         <plugin name="gazebo_ros_ackermann_drive" filename="libgazebo_ros_ackermann_drive.so">
-            <!-- ROS Namespace and Remappings -->
-            <ros>
-                <namespace>/</namespace> <!-- Set this to your robot's model name -->
-                <remapping>cmd_vel:=cmd_vel</remapping>
-                <remapping>odom:=odom</remapping>
-            </ros>
-            <!-- Update Rate -->
             <update_rate>100.0</update_rate>
-            <!-- Wheel Joints -->
+            <!-- wheels -->
             <front_left_joint>front_left_wheel_joint</front_left_joint>
             <front_right_joint>front_right_wheel_joint</front_right_joint>
             <rear_left_joint>rear_left_wheel_joint</rear_left_joint>
             <rear_right_joint>rear_right_wheel_joint</rear_right_joint>
-            <!-- Steering Joints -->
+            <!-- steering -->
             <left_steering_joint>left_steering_joint</left_steering_joint>
             <right_steering_joint>right_steering_joint</right_steering_joint>
-            <!-- Steering Limits -->
-            <max_steer>0.5</max_steer>
-            <!-- Max Steering Wheel Angle -->
+            <steering_wheel_joint>steering_wheel_joint</steering_wheel_joint>
+            <!-- Max absolute steer angle for tyre in radians-->
+            <!-- Any cmd_vel angular z greater than this would be capped -->
+            <max_steer>0.6458</max_steer>
+            <!-- Max absolute steering angle of steering wheel -->
             <max_steering_angle>7.85</max_steering_angle>
-            <!-- Max Speed -->
-            <max_speed>5.0</max_speed>
-            <!-- PID Tuning -->
-            <left_steering_pid_gain>500 0 50</left_steering_pid_gain>
+            <!-- Max absolute linear speed in m/s -->
+            <max_speed>20</max_speed>
+            <!-- PID tuning -->
+            <left_steering_pid_gain>1500 0 1</left_steering_pid_gain>
             <left_steering_i_range>0 0</left_steering_i_range>
-            <right_steering_pid_gain>500 0 50</right_steering_pid_gain>
+            <right_steering_pid_gain>1500 0 1</right_steering_pid_gain>
             <right_steering_i_range>0 0</right_steering_i_range>
-            <linear_velocity_pid_gain>300 10 20</linear_velocity_pid_gain>
-            <linear_velocity_i_range>-0.5 0.5</linear_velocity_i_range>
-            <!-- Output -->
+            <linear_velocity_pid_gain>1000 0 1</linear_velocity_pid_gain>
+            <linear_velocity_i_range>0 0</linear_velocity_i_range>
+            <!-- output -->
             <publish_odom>true</publish_odom>
             <publish_odom_tf>true</publish_odom_tf>
             <publish_wheel_tf>true</publish_wheel_tf>
-            <publish_distance>false</publish_distance>
-            <!-- Frames -->
+            <publish_distance>true</publish_distance>
             <odometry_frame>odom</odometry_frame>
-            <robot_base_frame>base_link</robot_base_frame>
-        </plugin>
-        <!-- Joint State Publisher Plugin -->
-        <plugin name="joint_state_publisher" filename="libgazebo_ros_joint_state_publisher.so">
-            <robotNamespace>/</robotNamespace> <!-- Set this to your robot's model name -->
-            <publishInterval>0.1</publishInterval>
-            <!-- List all joint names -->
-            <joint_name>front_left_wheel_joint</joint_name>
-            <joint_name>front_right_wheel_joint</joint_name>
-            <joint_name>rear_left_wheel_joint</joint_name>
-            <joint_name>rear_right_wheel_joint</joint_name>
-            <joint_name>left_steering_joint</joint_name>
-            <joint_name>right_steering_joint</joint_name>
+            <robot_base_frame>chassis</robot_base_frame>
         </plugin>
     </gazebo>

File: description/robot.urdf.xacro (robot description, xacro)
@@ -3,6 +3,8 @@
     <xacro:include filename="properties.xacro"/>
     <xacro:include filename="robot_core.xacro"/>
-    <xacro:include filename="gazebo_control.xacro"/>
+    <!---<xacro:include filename="gazebo_control.xacro"/>-->
     <xacro:include filename="lidar.xacro"/>
+    <xacro:include filename="camera.xacro"/>
+    <xacro:include filename="ros2_control.xacro"/>
     <!---<xacro:include filename="imu.xacro"/>-->
 </robot>

File: description/robot_core.xacro (robot description, xacro)
@@ -22,5 +22,4 @@
   <link name="chassis">
     <visual>
-      <origin xyz="0 0 0"/>
       <geometry>
         <box size="0.24 0.15 0.06"/>
@@ -29,5 +28,4 @@
     </visual>
     <collision>
-      <origin xyz="0 0 0"/>
       <geometry>
         <box size="0.24 0.15 0.06"/>
@@ -35,26 +33,26 @@
     </collision>
     <xacro:inertial_box mass="3.0" x="0.24" y="0.15" z="0.06">
-      <origin xyz="0 0 0"/>
+      <origin xyz="0 0 0" rpy="0 0 0"/>
     </xacro:inertial_box>
   </link>
-  <!-- Left Steering Joint -->
-  <joint name="left_steering_joint" type="revolute">
+  <!-- Central Rear Axle Joint -->
+  <joint name="rear_axle_joint" type="continuous">
     <parent link="chassis"/>
-    <child link="left_steering_link"/>
-    <origin xyz="0.12 0.09 -0.0375" rpy="1.5708 0 0"/>
-    <axis xyz="0 1 0"/>
-    <limit lower="-0.5" upper="0.5" effort="1000" velocity="1.0"/>
-  </joint>
-  <!-- Left Steering Link -->
-  <link name="left_steering_link"/>
-  <!-- Front Left Wheel Joint -->
-  <joint name="front_left_wheel_joint" type="continuous">
-    <parent link="left_steering_link"/>
-    <child link="front_left_wheel"/>
-    <origin xyz="0 0 0" rpy="0 0 0"/>
+    <child link="rear_axle_link"/>
+    <origin xyz="-0.12 0 0" rpy="0 0 0"/>
     <axis xyz="0 0 1"/>
   </joint>
-  <!-- Front Left Wheel Link -->
-  <link name="front_left_wheel">
+  <!-- Rear Axle Link -->
+  <link name="rear_axle_link"/>
+  <!-- Rear Left Wheel Joint (Mimics Central Axle) -->
+  <joint name="rear_left_wheel_joint" type="continuous">
+    <parent link="rear_axle_link"/>
+    <child link="rear_left_wheel"/>
+    <origin xyz="0.0 0.09 0" rpy="1.5708 0 0"/>
+    <axis xyz="0 0 1"/>
+    <mimic joint="rear_axle_joint" multiplier="1.0"/>
+  </joint>
+  <!-- Rear Left Wheel Link -->
+  <link name="rear_left_wheel">
     <visual>
       <geometry>
@@ -69,22 +67,71 @@
     </collision>
     <xacro:inertial_cylinder mass="0.1" length="0.025" radius="0.0375">
-      <origin xyz="0 0 0"/>
+      <origin xyz="0 0 0" rpy="0 0 0"/>
     </xacro:inertial_cylinder>
   </link>
-  <!-- Right Steering Joint -->
-  <joint name="right_steering_joint" type="revolute">
+  <!-- Rear Right Wheel Joint (Mimics Central Axle) -->
+  <joint name="rear_right_wheel_joint" type="continuous">
+    <parent link="rear_axle_link"/>
+    <child link="rear_right_wheel"/>
+    <origin xyz="0.0 -0.09 0" rpy="1.5708 0 0"/>
+    <axis xyz="0 0 1"/>
+    <mimic joint="rear_axle_joint" multiplier="1.0"/>
+  </joint>
+  <!-- Rear Right Wheel Link -->
+  <link name="rear_right_wheel">
+    <visual>
+      <geometry>
+        <cylinder radius="0.0375" length="0.025"/>
+      </geometry>
+      <material name="blue"/>
+    </visual>
+    <collision>
+      <geometry>
+        <cylinder radius="0.0375" length="0.025"/>
+      </geometry>
+    </collision>
+    <xacro:inertial_cylinder mass="0.1" length="0.025" radius="0.0375">
+      <origin xyz="0 0 0" rpy="0 0 0"/>
+    </xacro:inertial_cylinder>
+  </link>
+  <!-- Front Steering Joint -->
+  <joint name="front_steer_joint" type="revolute">
     <parent link="chassis"/>
-    <child link="right_steering_link"/>
-    <origin xyz="0.12 -0.09 -0.0375" rpy="1.5708 0 0"/>
+    <child link="steering_link"/>
+    <origin xyz="0.12 0 0.0375" rpy="1.5708 0 0"/>
     <axis xyz="0 1 0"/>
-    <limit lower="-0.5" upper="0.5" effort="1000" velocity="1.0"/>
+    <limit lower="-0.5" upper="0.5" effort="1000" velocity="5.0"/>
   </joint>
-  <!-- Right Steering Link -->
-  <link name="right_steering_link"/>
+  <!-- Steering Link -->
+  <link name="steering_link"/>
+  <!-- Front Left Wheel Joint -->
+  <joint name="front_left_wheel_joint" type="continuous">
+    <parent link="steering_link"/>
+    <child link="front_left_wheel"/>
+    <origin xyz="0.0 0.09 0"/>
+    <axis xyz="0 0 1"/>
+  </joint>
+  <!-- Front Left Wheel Link -->
+  <link name="front_left_wheel">
+    <visual>
+      <geometry>
+        <cylinder radius="0.0375" length="0.025"/>
+      </geometry>
+      <material name="orange"/>
+    </visual>
+    <collision>
+      <geometry>
+        <cylinder radius="0.0375" length="0.025"/>
+      </geometry>
+    </collision>
+    <xacro:inertial_cylinder mass="0.1" length="0.025" radius="0.0375">
+      <origin xyz="0 0 0" rpy="0 0 0"/>
+    </xacro:inertial_cylinder>
+  </link>
   <!-- Front Right Wheel Joint -->
   <joint name="front_right_wheel_joint" type="continuous">
-    <parent link="right_steering_link"/>
+    <parent link="steering_link"/>
     <child link="front_right_wheel"/>
-    <origin xyz="0 0 0" rpy="0 0 0"/>
+    <origin xyz="0.0 -0.09 0"/>
     <axis xyz="0 0 1"/>
   </joint>
@@ -103,53 +150,5 @@
     </collision>
     <xacro:inertial_cylinder mass="0.1" length="0.025" radius="0.0375">
-      <origin xyz="0 0 0"/>
-    </xacro:inertial_cylinder>
-  </link>
-  <!-- Rear Left Wheel Joint -->
-  <joint name="rear_left_wheel_joint" type="continuous">
-    <parent link="chassis"/>
-    <child link="rear_left_wheel"/>
-    <origin xyz="-0.12 0.09 -0.0375" rpy="1.5708 0 0"/>
-    <axis xyz="0 0 1"/>
-  </joint>
-  <!-- Rear Left Wheel Link -->
-  <link name="rear_left_wheel">
-    <visual>
-      <geometry>
-        <cylinder radius="0.0375" length="0.025"/>
-      </geometry>
-      <material name="blue"/>
-    </visual>
-    <collision>
-      <geometry>
-        <cylinder radius="0.0375" length="0.025"/>
-      </geometry>
-    </collision>
-    <xacro:inertial_cylinder mass="0.1" length="0.025" radius="0.0375">
-      <origin xyz="0 0 0"/>
-    </xacro:inertial_cylinder>
-  </link>
-  <!-- Rear Right Wheel Joint -->
-  <joint name="rear_right_wheel_joint" type="continuous">
-    <parent link="chassis"/>
-    <child link="rear_right_wheel"/>
-    <origin xyz="-0.12 -0.09 -0.0375" rpy="1.5708 0 0"/>
-    <axis xyz="0 0 1"/>
-  </joint>
-  <!-- Rear Right Wheel Link -->
-  <link name="rear_right_wheel">
-    <visual>
-      <geometry>
-        <cylinder radius="0.0375" length="0.025"/>
-      </geometry>
-      <material name="blue"/>
-    </visual>
-    <collision>
-      <geometry>
-        <cylinder radius="0.0375" length="0.025"/>
-      </geometry>
-    </collision>
-    <xacro:inertial_cylinder mass="0.1" length="0.025" radius="0.0375">
-      <origin xyz="0 0 0"/>
+      <origin xyz="0 0 0" rpy="0 0 0"/>
     </xacro:inertial_cylinder>
   </link>
@@ -174,5 +173,5 @@
     </collision>
     <xacro:inertial_box mass="0.05" x="0.025" y="0.09" z="0.02">
-      <origin xyz="0 0 0"/>
+      <origin xyz="0 0 0" rpy="0 0 0"/>
     </xacro:inertial_box>
   </link>

File: description/ros2_control.xacro (robot description, xacro)
@@ -1,28 +1,35 @@
 <?xml version="1.0"?>
-<robot xmlns:xacro="http://www.ros.org/wiki/xacro" >
-    <ros2_control name="GazeboSystem" type="system">
+<robot xmlns:xacro="http://www.ros.org/wiki/xacro">
+    <ros2_control name="AckermannSteeringSystem" type="system">
         <hardware>
             <plugin>gazebo_ros2_control/GazeboSystem</plugin>
         </hardware>
-        <joint name="left_wheel_joint">
-            <command_interface name="velocity">
-                <param name="min">-10</param>
-                <param name="max">10</param>
-            </command_interface>
+        <!-- Front Steering Joint -->
+        <joint name="front_steer_joint">
+            <command_interface name="position"/>
+            <state_interface name="position"/>
+        </joint>
+        <!-- Rear Axle Joint -->
+        <joint name="rear_axle_joint">
+            <command_interface name="velocity"/>
             <state_interface name="velocity"/>
             <state_interface name="position"/>
         </joint>
-        <joint name="right_wheel_joint">
-            <command_interface name="velocity">
-                <param name="min">-10</param>
-                <param name="max">10</param>
-            </command_interface>
+        <!-- Rear Left Wheel (Mimicking Rear Axle) -->
+        <joint name="rear_left_wheel_joint">
+            <command_interface name="velocity"/>
             <state_interface name="velocity"/>
-            <state_interface name="position"/>
+            <mimic joint="rear_axle_joint" multiplier="1.0"/>
+        </joint>
+        <!-- Rear Right Wheel (Mimicking Rear Axle) -->
+        <joint name="rear_right_wheel_joint">
+            <command_interface name="velocity"/>
+            <state_interface name="velocity"/>
+            <mimic joint="rear_axle_joint" multiplier="1.0"/>
         </joint>
     </ros2_control>
     <gazebo>
         <plugin name="gazebo_ros2_control" filename="libgazebo_ros2_control.so">
-            <parameters>$(find f112th_sim_2402_bravo)/config/my_controllers.yaml</parameters>
+            <parameters>/home/d/ros2_ws_2402/install/f112th_sim_2402_bravo/share/f112th_sim_2402_bravo/config/my_controllers.yaml</parameters>
         </plugin>
     </gazebo>
